File: pcb/intex-swg-pcb.kicad_pcb (KiCad board)
At the start: 2 copper layers, 70.2 x 90 mm, 12 parts, among them J1 230V, J2 Relay Board, J3 Display Board, J4 Main Board

Commit message: Swapped relay to GPIO2
Connections:
- MD1 pad 24: Net-(MD1-Pad24) -> /RELAY
- MD1 pad 25: /RELAY -> Net-(MD1-Pad25)
Routing:
- net /RELAY: track 25.0 -> 22.6 mm
